File: eagle/akcel_onlyboard.brd (EAGLE design)
At the start: 40.3 x 49.5 mm, 12 parts

Commit message: Poprawiono troszku płytkę
Routing:
- net N$14: track 29.2 -> 1.27 mm
- net N$3: track 14.0 -> 0.00 mm
- net N$18: track 11.7 -> 0.00 mm
- net N$17: track 7.44 -> 0.00 mm
- net N$13: track 6.35 -> 0.00 mm
- net N$12: track 6.35 -> 0.00 mm
- net N$10: track 6.35 -> 0.00 mm
- net N$15: track 5.31 -> 0.00 mm
- net N$16: track 3.81 -> 0.00 mm
Changed lines of the file:
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@@
 <wire x1="5.8064" y1="20.32" x2="5.9334" y2="20.193" width="0.8128" layer="1"/>
 </signal>
-<signal name="N$3">
-<wire x1="16.51" y1="10.16" x2="13.97" y2="10.16" width="1.27" layer="1"/>
-<wire x1="13.97" y1="10.16" x2="13.97" y2="11.43" width="1.27" layer="1"/>
-<wire x1="13.97" y1="11.43" x2="16.51" y2="11.43" width="1.27" layer="1"/>
-<wire x1="16.51" y1="11.43" x2="16.51" y2="10.16" width="1.27" layer="1"/>
-<wire x1="16.51" y1="10.16" x2="16.51" y2="6.35" width="1.27" layer="1"/>
-<wire x1="16.51" y1="6.35" x2="15.24" y2="6.35" width="1.27" layer="1"/>
-<wire x1="16.51" y1="6.35" x2="17.78" y2="6.35" width="1.27" layer="1"/>
-</signal>
-<signal name="N$10">
-<wire x1="22.86" y1="6.35" x2="22.86" y2="3.81" width="1.27" layer="1"/>
-<wire x1="22.86" y1="3.81" x2="21.59" y2="3.81" width="1.27" layer="1"/>
-<wire x1="21.59" y1="3.81" x2="21.59" y2="6.35" width="1.27" layer="1"/>
-</signal>
-<signal name="N$12">
-<wire x1="3.81" y1="7.62" x2="6.35" y2="7.62" width="1.27" layer="1"/>
-<wire x1="6.35" y1="7.62" x2="6.35" y2="6.35" width="1.27" layer="1"/>
-<wire x1="6.35" y1="6.35" x2="3.81" y2="6.35" width="1.27" layer="1"/>
-</signal>
-<signal name="N$13">
-<wire x1="3.81" y1="3.81" x2="6.35" y2="3.81" width="1.27" layer="1"/>
-<wire x1="6.35" y1="3.81" x2="6.35" y2="2.54" width="1.27" layer="1"/>
-<wire x1="6.35" y1="2.54" x2="3.81" y2="2.54" width="1.27" layer="1"/>
-</signal>
 <signal name="N$14">
-<wire x1="1.27" y1="13.97" x2="0" y2="13.97" width="1.27" layer="1"/>
-<wire x1="0" y1="13.97" x2="0" y2="15.24" width="1.27" layer="1"/>
-<wire x1="0" y1="15.24" x2="1.27" y2="15.24" width="1.27" layer="1"/>
-<wire x1="1.27" y1="15.24" x2="1.27" y2="16.51" width="1.27" layer="1"/>
-<wire x1="1.27" y1="16.51" x2="0" y2="16.51" width="1.27" layer="1"/>
-<wire x1="0" y1="16.51" x2="0" y2="12.7" width="1.27" layer="1"/>
-<wire x1="0" y1="12.7" x2="1.27" y2="12.7" width="1.27" layer="1"/>
-<wire x1="1.27" y1="12.7" x2="1.27" y2="11.43" width="1.27" layer="1"/>
-<wire x1="1.27" y1="11.43" x2="0" y2="11.43" width="1.27" layer="1"/>
-<wire x1="1.27" y1="11.43" x2="3.81" y2="11.43" width="1.27" layer="1"/>
-<wire x1="3.81" y1="11.43" x2="3.81" y2="12.7" width="1.27" layer="1"/>
 <wire x1="3.81" y1="15.24" x2="2.54" y2="15.24" width="1.27" layer="1"/>
-<wire x1="2.54" y1="15.24" x2="2.54" y2="16.51" width="1.27" layer="1"/>
-<wire x1="2.54" y1="16.51" x2="1.27" y2="16.51" width="1.27" layer="1"/>
-<wire x1="2.54" y1="16.51" x2="3.81" y2="16.51" width="1.27" layer="1"/>
-<wire x1="3.81" y1="16.51" x2="3.81" y2="17.78" width="1.27" layer="1"/>
-<wire x1="3.81" y1="16.51" x2="3.81" y2="15.24" width="1.27" layer="1"/>
-<wire x1="3.81" y1="15.24" x2="3.81" y2="12.7" width="1.27" layer="1"/>
-<wire x1="3.81" y1="11.43" x2="3.81" y2="10.16" width="1.27" layer="1"/>
-</signal>
-<signal name="N$15">
-<wire x1="-1.27" y1="21.59" x2="-1.27" y2="19.05" width="1.27" layer="1"/>
-<wire x1="-1.27" y1="19.05" x2="-0.6604" y2="19.05" width="1.27" layer="1"/>
-<wire x1="-0.6604" y1="19.05" x2="-0.6604" y2="19.2532" width="1.27" layer="1"/>
-<wire x1="-0.6604" y1="19.2532" x2="-0.6096" y2="19.2532" width="1.27" layer="1"/>
-<wire x1="-0.6096" y1="19.2532" x2="-0.6096" y2="21.1582" width="1.27" layer="1"/>
-</signal>
-<signal name="N$16">
-<wire x1="19.05" y1="12.7" x2="21.59" y2="12.7" width="1.27" layer="1"/>
-<wire x1="21.59" y1="12.7" x2="21.59" y2="11.43" width="1.27" layer="1"/>
-</signal>
-<signal name="N$17">
-<wire x1="-0.4826" y1="39.8018" x2="-0.1778" y2="39.8018" width="1.27" layer="1"/>
-<wire x1="-0.1778" y1="39.8018" x2="-0.1778" y2="39.7764" width="1.27" layer="1"/>
-<wire x1="-0.1778" y1="39.7764" x2="2.8956" y2="39.7764" width="1.27" layer="1"/>
-<wire x1="2.8956" y1="39.7764" x2="2.8956" y2="39.8526" width="1.27" layer="1"/>
-<wire x1="2.8956" y1="39.8526" x2="2.6924" y2="39.8526" width="1.27" layer="1"/>
-<wire x1="2.6924" y1="39.8526" x2="2.6924" y2="38.9382" width="1.27" layer="1"/>
-<wire x1="2.6924" y1="38.9382" x2="-0.1524" y2="38.9382" width="1.27" layer="1"/>
-</signal>
-<signal name="N$18">
-<wire x1="-0.9652" y1="26.797" x2="2.9718" y2="26.797" width="1.27" layer="1"/>
-<wire x1="2.9718" y1="26.797" x2="2.9718" y2="26.6192" width="1.27" layer="1"/>
-<wire x1="2.9718" y1="26.6192" x2="2.7178" y2="26.6192" width="1.27" layer="1"/>
-<wire x1="2.7178" y1="26.6192" x2="2.7178" y2="27.1526" width="1.27" layer="1"/>
-<wire x1="2.7178" y1="27.1526" x2="-0.127" y2="27.1526" width="1.27" layer="1"/>
-<wire x1="-0.127" y1="27.1526" x2="-0.127" y2="27.0002" width="1.27" layer="1"/>
-<wire x1="-0.127" y1="27.0002" x2="-0.254" y2="27.0002" width="1.27" layer="1"/>
-<wire x1="-0.254" y1="27.0002" x2="-0.254" y2="26.1874" width="1.27" layer="1"/>
-<wire x1="-0.254" y1="26.1874" x2="2.5146" y2="26.1874" width="1.27" layer="1"/>
-<wire x1="2.5146" y1="26.1874" x2="2.5146" y2="26.3144" width="1.27" layer="1"/>
 </signal>
 </signals>
