File: eagle/akcel.sch (EAGLE design)
At the start: 23 parts, among them CON1 MINI-USB, IC1 TP4056, SW1 CT10-XXXX-A2, U1 GY-521MPU6050

Commit message: Dodano pracke
Parts:
- LI-ION: value 3.6V -> 3.8V
Connections:
- net 5V: no longer C4.1, IC1.BAT
- net BAT+: now also C4.1, IC1.BAT
Changed lines of the file:
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@@
 <part name="C2" library="rcl" deviceset="CPOL-EU" device="085CS-1AR" value="2.2uF"/>
 <part name="C3" library="rcl" deviceset="C-EU" device="025-024X044" value="100nF"/>
-<part name="LI-ION" library="special" deviceset="BATTERY" device="" value="3.6V"/>
+<part name="LI-ION" library="special" deviceset="BATTERY" device="" value="3.8V"/>
 <part name="LED1" library="led" deviceset="LED" device="10MM"/>
 <part name="R1" library="rcl" deviceset="R-EU_" device="0204/2V" value="10k"/>
@@
 <label x="27.94" y="104.14" size="1.778" layer="95" rot="R180" xref="yes"/>
 </segment>
+<segment>
+<pinref part="IC1" gate="G$1" pin="BAT"/>
+<wire x1="73.66" y1="142.24" x2="81.28" y2="142.24" width="0.1524" layer="91"/>
+<pinref part="C4" gate="G$1" pin="1"/>
+<wire x1="81.28" y1="142.24" x2="81.28" y2="139.7" width="0.1524" layer="91"/>
+<wire x1="81.28" y1="142.24" x2="81.28" y2="170.18" width="0.1524" layer="91"/>
+<junction x="81.28" y="142.24"/>
+<label x="81.28" y="170.18" size="1.778" layer="95" rot="R90" xref="yes"/>
+</segment>
 </net>
 <net name="N$6" class="0">
@@
 </segment>
 <segment>
-<pinref part="IC1" gate="G$1" pin="BAT"/>
-<wire x1="73.66" y1="142.24" x2="81.28" y2="142.24" width="0.1524" layer="91"/>
-<pinref part="C4" gate="G$1" pin="1"/>
-<wire x1="81.28" y1="142.24" x2="81.28" y2="139.7" width="0.1524" layer="91"/>
-<wire x1="81.28" y1="142.24" x2="81.28" y2="172.72" width="0.1524" layer="91"/>
-<junction x="81.28" y="142.24"/>
-<label x="81.28" y="172.72" size="1.778" layer="95" rot="R90" xref="yes"/>
-</segment>
-<segment>
